Commit message: Split lidar, dock connector and casters out of body mesh
The laser_frame sat inside the merged body.stl, so scan rays and collision
checks hit the body. Separate the parts so each can have its own visual and
collision:

- lidar.stl: visual on laser_frame, no collision (ray sensors ignore it)
- docking.stl: static connector, visual on base_link
- solenoid.stl: lifted 0.0735 so its top is flush with the connector at
  docking_joint=0; collision/inertia now match the sleeve
- caster_l/r.stl: new fixed links with r=0.0153 sphere collisions
- base_link collision box raised to z 0.0075-0.095 so only wheels and
  casters touch the ground

File: ros2/kachaka_description/urdf/_kachaka.urdf.xacro (robot description, xacro)
@@ -25,9 +25,18 @@
         <material name="body" />
       </visual>
-      <collision>
-        <origin xyz="0.0435 0.0 0.0475"
-                rpy="0 0 0" />
-        <geometry>
-          <box size="0.387 0.240 0.095" />
+      <!-- Static dock connector split from body.stl; mesh is in base_link coords -->
+      <visual>
+        <origin rpy="0 0 0" xyz="0 0 0"/>
+        <geometry>
+          <mesh filename="file://$(find kachaka_description)/meshes/kachaka/docking.stl"/>
+        </geometry>
+        <material name="body" />
+      </visual>
+      <!-- Spans body underside (z=0.0075) to top plate (z=0.095); only wheels and casters touch ground -->
+      <collision>
+        <origin xyz="0.0435 0.0 ${(0.0075 + 0.095) / 2}"
+                rpy="0 0 0" />
+        <geometry>
+          <box size="0.387 0.240 ${0.095 - 0.0075}" />
         </geometry>
         <material name="body" />
@@ -113,4 +122,52 @@
       </collision>
     </link>
+    <!-- Caster(right) split from body.stl; mesh origin at ball centre, ball rests on z=0 -->
+    <joint name="base_r_caster_joint"
+          type="fixed">
+      <parent link="base_link" />
+      <child link="base_r_caster_link" />
+      <origin rpy="0 0 0"
+              xyz="0.1945 -0.0678 0.0153" />
+    </joint>
+    <link name="base_r_caster_link">
+      <visual>
+        <origin rpy="0 0 0" xyz="0 0 0"/>
+        <geometry>
+          <mesh filename="file://$(find kachaka_description)/meshes/kachaka/caster_r.stl"/>
+        </geometry>
+        <material name="tire" />
+      </visual>
+      <collision>
+        <origin xyz="0 0 0"
+                rpy="0 0 0" />
+        <geometry>
+          <sphere radius="0.0153" />
+        </geometry>
+      </collision>
+    </link>
+    <!-- Caster(left) split from body.stl; mesh origin at ball centre, ball rests on z=0 -->
+    <joint name="base_l_caster_joint"
+          type="fixed">
+      <parent link="base_link" />
+      <child link="base_l_caster_link" />
+      <origin rpy="0 0 0"
+              xyz="0.1971 0.0796 0.0153" />
+    </joint>
+    <link name="base_l_caster_link">
+      <visual>
+        <origin rpy="0 0 0" xyz="0 0 0"/>
+        <geometry>
+          <mesh filename="file://$(find kachaka_description)/meshes/kachaka/caster_l.stl"/>
+        </geometry>
+        <material name="tire" />
+      </visual>
+      <collision>
+        <origin xyz="0 0 0"
+                rpy="0 0 0" />
+        <geometry>
+          <sphere radius="0.0153" />
+        </geometry>
+      </collision>
+    </link>
     <!-- 2D LiDAR -->
     <joint name="lidar_joint"
@@ -121,5 +178,14 @@
               xyz="0.156 0 0.1049" />
     </joint>
-    <link name="laser_frame" />
+    <!-- LiDAR head split from body.stl so scan-plane hits can be tuned per sim; mesh is in laser_frame coords -->
+    <link name="laser_frame">
+      <visual>
+        <origin rpy="0 0 0" xyz="0 0 0"/>
+        <geometry>
+          <mesh filename="file://$(find kachaka_description)/meshes/kachaka/lidar.stl"/>
+        </geometry>
+        <material name="body" />
+      </visual>
+    </link>
     <!-- Camera(front) -->
     <joint name="camera_front_joint"
@@ -165,11 +231,13 @@
       <inertial>
         <mass value="0.2" /> <!-- TODO - Update mass value -->
-        <origin xyz="0 0 0.1075"
-                rpy="0 0 0" />
-        <inertia ixx="${1/12*0.2*(3*0.025**2+0.015**2)}" ixy="0" ixz="0"
-                 iyy="${1/12*0.2*(3*0.025**2+0.015**2)}" iyz="0"
-                 izz="${1/2*0.2*(0.025**2)}" />
-      </inertial>
-      <visual>
+        <origin xyz="0 0 ${0.0735 + 0.0395 / 2}"
+                rpy="0 0 0" />
+        <inertia ixx="${1/12*0.2*(3*0.030**2+0.0395**2)}" ixy="0" ixz="0"
+                 iyy="${1/12*0.2*(3*0.030**2+0.0395**2)}" iyz="0"
+                 izz="${1/2*0.2*(0.030**2)}" />
+      </inertial>
+      <!-- solenoid.stl spans z 0..0.0395; lift so its top meets the connector top (z=0.113) -->
+      <visual>
+        <origin rpy="0 0 0" xyz="0 0 0.0735"/>
         <geometry>
           <mesh filename="file://$(find kachaka_description)/meshes/kachaka/solenoid.stl"
@@ -179,9 +247,9 @@
       </visual>
       <collision>
-        <origin xyz="0 0 0.1075"
-                rpy="0 0 0" />
-        <geometry>
-          <cylinder length="0.015"
-                    radius="0.025" />
+        <origin xyz="0 0 ${0.0735 + 0.0395 / 2}"
+                rpy="0 0 0" />
+        <geometry>
+          <cylinder length="0.0395"
+                    radius="0.030" />
         </geometry>
         <material name="body" />

Commit message: Add placeholder inertial to laser_frame
A link with a visual but no inertial gets a default 1 kg in Isaac/PhysX.

File: ros2/kachaka_description/urdf/_kachaka.urdf.xacro (robot description, xacro)
@@ -187,4 +187,13 @@
         <material name="body" />
       </visual>
+      <!-- Tiny placeholder; without it Isaac/PhysX gives a visual-only link a default 1 kg -->
+      <inertial>
+        <mass value="0.001" />
+        <origin xyz="0 0 0"
+                rpy="0 0 0" />
+        <inertia ixx="1e-7" ixy="0" ixz="0"
+                 iyy="1e-7" iyz="0"
+                 izz="1e-7" />
+      </inertial>
     </link>
     <!-- Camera(front) -->
